Commit message: Release v2026.7.14

File: hand/body-with-soft/urdf/left-ros.urdf (robot description, URDF)
Before this commit: robot wujihand-left, 27 links, 26 joints
Links:
- link left_finger1_link1: geometry collision mesh filename=package://wuji_description/body-with-soft/meshes/left/left_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; visual mesh filename=package://wuji_description/body-with-soft/meshes/left/left_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
- link left_finger1_link2: geometry collision mesh filename=package://wuji_description/body-with-soft/meshes/left/left_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; visual mesh filename=package://wuji_description/body-with-soft/meshes/left/left_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
- link left_finger1_link2_softbody: geometry collision mesh filename=package://wuji_description/body-with-soft/meshes/left/left_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; visual mesh filename=package://wuji_description/body-with-soft/meshes/left/left_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
- link left_finger1_link3: geometry collision mesh filename=package://wuji_description/body-with-soft/meshes/left/left_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; visual mesh filename=package://wuji_description/body-with-soft/meshes/left/left_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
- link left_finger1_link4: geometry collision mesh filename=package://wuji_description/body-with-soft/meshes/left/left_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; visual mesh filename=package://wuji_description/body-with-soft/meshes/left/left_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
- link left_finger1_tip_link: geometry collision mesh filename=package://wuji_description/body-with-soft/meshes/left/left_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; visual mesh filename=package://wuji_description/body-with-soft/meshes/left/left_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
- link left_finger2_link1: geometry collision mesh filename=package://wuji_description/body-with-soft/meshes/left/left_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; visual mesh filename=package://wuji_description/body-with-soft/meshes/left/left_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
- link left_finger2_link2: geometry collision mesh filename=package://wuji_description/body-with-soft/meshes/left/left_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; visual mesh filename=package://wuji_description/body-with-soft/meshes/left/left_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
- link left_finger2_link3: geometry collision mesh filename=package://wuji_description/body-with-soft/meshes/left/left_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; visual mesh filename=package://wuji_description/body-with-soft/meshes/left/left_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
- link left_finger2_link4: geometry collision mesh filename=package://wuji_description/body-with-soft/meshes/left/left_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; visual mesh filename=package://wuji_description/body-with-soft/meshes/left/left_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
- link left_finger2_tip_link: geometry collision mesh filename=package://wuji_description/body-with-soft/meshes/left/left_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; visual mesh filename=package://wuji_description/body-with-soft/meshes/left/left_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
- link left_finger3_link1: geometry collision mesh filename=package://wuji_description/body-with-soft/meshes/left/left_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; visual mesh filename=package://wuji_description/body-with-soft/meshes/left/left_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
- link left_finger3_link2: geometry collision mesh filename=package://wuji_description/body-with-soft/meshes/left/left_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; visual mesh filename=package://wuji_description/body-with-soft/meshes/left/left_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
- link left_finger3_link3: geometry collision mesh filename=package://wuji_description/body-with-soft/meshes/left/left_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; visual mesh filename=package://wuji_description/body-with-soft/meshes/left/left_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
- link left_finger3_link4: geometry collision mesh filename=package://wuji_description/body-with-soft/meshes/left/left_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; visual mesh filename=package://wuji_description/body-with-soft/meshes/left/left_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
- link left_finger3_tip_link: geometry collision mesh filename=package://wuji_description/body-with-soft/meshes/left/left_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; visual mesh filename=package://wuji_description/body-with-soft/meshes/left/left_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
- link left_finger4_link1: geometry collision mesh filename=package://wuji_description/body-with-soft/meshes/left/left_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; visual mesh filename=package://wuji_description/body-with-soft/meshes/left/left_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
- link left_finger4_link2: geometry collision mesh filename=package://wuji_description/body-with-soft/meshes/left/left_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; visual mesh filename=package://wuji_description/body-with-soft/meshes/left/left_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
- link left_finger4_link3: geometry collision mesh filename=package://wuji_description/body-with-soft/meshes/left/left_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; visual mesh filename=package://wuji_description/body-with-soft/meshes/left/left_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
- link left_finger4_link4: geometry collision mesh filename=package://wuji_description/body-with-soft/meshes/left/left_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; visual mesh filename=package://wuji_description/body-with-soft/meshes/left/left_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
- link left_finger4_tip_link: geometry collision mesh filename=package://wuji_description/body-with-soft/meshes/left/left_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; visual mesh filename=package://wuji_description/body-with-soft/meshes/left/left_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
- link left_finger5_link1: geometry collision mesh filename=package://wuji_description/body-with-soft/meshes/left/left_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; visual mesh filename=package://wuji_description/body-with-soft/meshes/left/left_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
- link left_finger5_link2: geometry collision mesh filename=package://wuji_description/body-with-soft/meshes/left/left_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; visual mesh filename=package://wuji_description/body-with-soft/meshes/left/left_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
- link left_finger5_link3: geometry collision mesh filename=package://wuji_description/body-with-soft/meshes/left/left_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; visual mesh filename=package://wuji_description/body-with-soft/meshes/left/left_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
- link left_finger5_link4: geometry collision mesh filename=package://wuji_description/body-with-soft/meshes/left/left_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; visual mesh filename=package://wuji_description/body-with-soft/meshes/left/left_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
- link left_finger5_tip_link: geometry collision mesh filename=package://wuji_description/body-with-soft/meshes/left/left_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; visual mesh filename=package://wuji_description/body-with-soft/meshes/left/left_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
- link left_palm_link: geometry collision mesh filename=package://wuji_description/body-with-soft/meshes/left/left_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; visual mesh filename=package://wuji_description/body-with-soft/meshes/left/left_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

File: hand/body-with-soft/urdf/right-ros.urdf (robot description, URDF)
Before this commit: robot wujihand-right, 27 links, 26 joints
Links:
- link right_finger1_link1: geometry collision mesh filename=package://wuji_description/body-with-soft/meshes/right/righ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; visual mesh filename=package://wuji_description/body-with-soft/meshes/right/righ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
- link right_finger1_link2: geometry collision mesh filename=package://wuji_description/body-with-soft/meshes/right/righ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; visual mesh filename=package://wuji_description/body-with-soft/meshes/right/righ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
- link right_finger1_link2_softbody: geometry collision mesh filename=package://wuji_description/body-with-soft/meshes/right/righ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; visual mesh filename=package://wuji_description/body-with-soft/meshes/right/righ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
- link right_finger1_link3: geometry collision mesh filename=package://wuji_description/body-with-soft/meshes/right/righ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; visual mesh filename=package://wuji_description/body-with-soft/meshes/right/righ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
- link right_finger1_link4: geometry collision mesh filename=package://wuji_description/body-with-soft/meshes/right/righ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; visual mesh filename=package://wuji_description/body-with-soft/meshes/right/righ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
- link right_finger1_tip_link: geometry collision mesh filename=package://wuji_description/body-with-soft/meshes/right/righ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; visual mesh filename=package://wuji_description/body-with-soft/meshes/right/righ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
- link right_finger2_link1: geometry collision mesh filename=package://wuji_description/body-with-soft/meshes/right/righ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; visual mesh filename=package://wuji_description/body-with-soft/meshes/right/righ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
- link right_finger2_link2: geometry collision mesh filename=package://wuji_description/body-with-soft/meshes/right/righ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; visual mesh filename=package://wuji_description/body-with-soft/meshes/right/righ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
- link right_finger2_link3: geometry collision mesh filename=package://wuji_description/body-with-soft/meshes/right/righ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; visual mesh filename=package://wuji_description/body-with-soft/meshes/right/righ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
- link right_finger2_link4: geometry collision mesh filename=package://wuji_description/body-with-soft/meshes/right/righ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; visual mesh filename=package://wuji_description/body-with-soft/meshes/right/righ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
- link right_finger2_tip_link: geometry collision mesh filename=package://wuji_description/body-with-soft/meshes/right/righ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; visual mesh filename=package://wuji_description/body-with-soft/meshes/right/righ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
- link right_finger3_link1: geometry collision mesh filename=package://wuji_description/body-with-soft/meshes/right/righ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; visual mesh filename=package://wuji_description/body-with-soft/meshes/right/righ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
- link right_finger3_link2: geometry collision mesh filename=package://wuji_description/body-with-soft/meshes/right/righ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; visual mesh filename=package://wuji_description/body-with-soft/meshes/right/righ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
- link right_finger3_link3: geometry collision mesh filename=package://wuji_description/body-with-soft/meshes/right/righ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; visual mesh filename=package://wuji_description/body-with-soft/meshes/right/righ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
- link right_finger3_link4: geometry collision mesh filename=package://wuji_description/body-with-soft/meshes/right/righ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; visual mesh filename=package://wuji_description/body-with-soft/meshes/right/righ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
- link right_finger3_tip_link: geometry collision mesh filename=package://wuji_description/body-with-soft/meshes/right/righ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; visual mesh filename=package://wuji_description/body-with-soft/meshes/right/righ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
- link right_finger4_link1: geometry collision mesh filename=package://wuji_description/body-with-soft/meshes/right/righ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; visual mesh filename=package://wuji_description/body-with-soft/meshes/right/righ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
- link right_finger4_link2: geometry collision mesh filename=package://wuji_description/body-with-soft/meshes/right/righ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; visual mesh filename=package://wuji_description/body-with-soft/meshes/right/righ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
- link right_finger4_link3: geometry collision mesh filename=package://wuji_description/body-with-soft/meshes/right/righ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; visual mesh filename=package://wuji_description/body-with-soft/meshes/right/righ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
- link right_finger4_link4: geometry collision mesh filename=package://wuji_description/body-with-soft/meshes/right/righ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; visual mesh filename=package://wuji_description/body-with-soft/meshes/right/righ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
- link right_finger4_tip_link: geometry collision mesh filename=package://wuji_description/body-with-soft/meshes/right/righ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; visual mesh filename=package://wuji_description/body-with-soft/meshes/right/righ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
- link right_finger5_link1: geometry collision mesh filename=package://wuji_description/body-with-soft/meshes/right/righ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; visual mesh filename=package://wuji_description/body-with-soft/meshes/right/righ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
- link right_finger5_link2: geometry collision mesh filename=package://wuji_description/body-with-soft/meshes/right/righ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; visual mesh filename=package://wuji_description/body-with-soft/meshes/right/righ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
- link right_finger5_link3: geometry collision mesh filename=package://wuji_description/body-with-soft/meshes/right/righ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; visual mesh filename=package://wuji_description/body-with-soft/meshes/right/righ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
- link right_finger5_link4: geometry collision mesh filename=package://wuji_description/body-with-soft/meshes/right/righ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; visual mesh filename=package://wuji_description/body-with-soft/meshes/right/righ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
- link right_finger5_tip_link: geometry collision mesh filename=package://wuji_description/body-with-soft/meshes/right/righ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; visual mesh filename=package://wuji_description/body-with-soft/meshes/right/righ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
- link right_palm_link: geometry collision mesh filename=package://wuji_description/body-with-soft/meshes/right/righ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; visual mesh filename=package://wuji_description/body-with-soft/meshes/right/righ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

File: hand2_beta/body/urdf/left-ros.urdf (robot description, URDF)
Before this commit: robot wujihand-left, 27 links, 26 joints
Links:
- link l_base_link: geometry collision mesh filename=package://wuji_description/hand2_beta/body/meshes/left/l_ba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; visual mesh filename=package://wuji_description/hand2_beta/body/meshes/left/l_ba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
- link l_index_finger_distal: geometry collision mesh filename=package://wuji_description/hand2_beta/body/meshes/left/l_in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; visual mesh filename=package://wuji_description/hand2_beta/body/meshes/left/l_in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
- link l_index_finger_middle: geometry collision mesh filename=package://wuji_description/hand2_beta/body/meshes/left/l_in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; visual mesh filename=package://wuji_description/hand2_beta/body/meshes/left/l_in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
- link l_index_finger_proximal: geometry collision mesh filename=package://wuji_description/hand2_beta/body/meshes/left/l_in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; visual mesh filename=package://wuji_description/hand2_beta/body/meshes/left/l_in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
- link l_index_finger_proximal_abd: geometry collision mesh filename=package://wuji_description/hand2_beta/body/meshes/left/l_in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; visual mesh filename=package://wuji_description/hand2_beta/body/meshes/left/l_in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
- link l_middle_finger_distal: geometry collision mesh filename=package://wuji_description/hand2_beta/body/meshes/left/l_mi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; visual mesh filename=package://wuji_description/hand2_beta/body/meshes/left/l_mi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
- link l_middle_finger_middle: geometry collision mesh filename=package://wuji_description/hand2_beta/body/meshes/left/l_mi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; visual mesh filename=package://wuji_description/hand2_beta/body/meshes/left/l_mi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
- link l_middle_finger_proximal: geometry collision mesh filename=package://wuji_description/hand2_beta/body/meshes/left/l_mi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; visual mesh filename=package://wuji_description/hand2_beta/body/meshes/left/l_mi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
- link l_middle_finger_proximal_abd: geometry collision mesh filename=package://wuji_description/hand2_beta/body/meshes/left/l_mi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; visual mesh filename=package://wuji_description/hand2_beta/body/meshes/left/l_mi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
- link l_pinky_distal: geometry collision mesh filename=package://wuji_description/hand2_beta/body/meshes/left/l_pi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; visual mesh filename=package://wuji_description/hand2_beta/body/meshes/left/l_pi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
- link l_pinky_middle: geometry collision mesh filename=package://wuji_description/hand2_beta/body/meshes/left/l_pi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; visual mesh filename=package://wuji_description/hand2_beta/body/meshes/left/l_pi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
- link l_pinky_proximal: geometry collision mesh filename=package://wuji_description/hand2_beta/body/meshes/left/l_pi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; visual mesh filename=package://wuji_description/hand2_beta/body/meshes/left/l_pi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
- link l_pinky_proximal_abd: geometry collision mesh filename=package://wuji_description/hand2_beta/body/meshes/left/l_pi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; visual mesh filename=package://wuji_description/hand2_beta/body/meshes/left/l_pi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
- link l_ring_finger_distal: geometry collision mesh filename=package://wuji_description/hand2_beta/body/meshes/left/l_ri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; visual mesh filename=package://wuji_description/hand2_beta/body/meshes/left/l_ri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
- link l_ring_finger_middle: geometry collision mesh filename=package://wuji_description/hand2_beta/body/meshes/left/l_ri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; visual mesh filename=package://wuji_description/hand2_beta/body/meshes/left/l_ri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
- link l_ring_finger_proximal: geometry collision mesh filename=package://wuji_description/hand2_beta/body/meshes/left/l_ri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; visual mesh filename=package://wuji_description/hand2_beta/body/meshes/left/l_ri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
- link l_ring_finger_proximal_abd: geometry collision mesh filename=package://wuji_description/hand2_beta/body/meshes/left/l_ri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; visual mesh filename=package://wuji_description/hand2_beta/body/meshes/left/l_ri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
- link l_thumb_distal: geometry collision mesh filename=package://wuji_description/hand2_beta/body/meshes/left/l_th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; visual mesh filename=package://wuji_description/hand2_beta/body/meshes/left/l_th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
- link l_thumb_middle: geometry collision mesh filename=package://wuji_description/hand2_beta/body/meshes/left/l_th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; visual mesh filename=package://wuji_description/hand2_beta/body/meshes/left/l_th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
- link l_thumb_proximal: geometry collision mesh filename=package://wuji_description/hand2_beta/body/meshes/left/l_th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; visual mesh filename=package://wuji_description/hand2_beta/body/meshes/left/l_th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
- link l_thumb_proximal_abd: geometry collision mesh filename=package://wuji_description/hand2_beta/body/meshes/left/l_th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; visual mesh filename=package://wuji_description/hand2_beta/body/meshes/left/l_th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
- link l_wrist: geometry collision mesh filename=package://wuji_description/hand2_beta/body/meshes/left/l_wr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; visual mesh filename=package://wuji_description/hand2_beta/body/meshes/left/l_wr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

File: hand2_beta/body/urdf/right-ros.urdf (robot description, URDF)
Before this commit: robot wujihand-right, 27 links, 26 joints
Links:
- link r_base_link: geometry collision mesh filename=package://wuji_description/hand2_beta/body/meshes/right/r_b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; visual mesh filename=package://wuji_description/hand2_beta/body/meshes/right/r_b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
- link r_index_finger_distal: geometry collision mesh filename=package://wuji_description/hand2_beta/body/meshes/right/r_i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; visual mesh filename=package://wuji_description/hand2_beta/body/meshes/right/r_i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
- link r_index_finger_middle: geometry collision mesh filename=package://wuji_description/hand2_beta/body/meshes/right/r_i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; visual mesh filename=package://wuji_description/hand2_beta/body/meshes/right/r_i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
- link r_index_finger_proximal: geometry collision mesh filename=package://wuji_description/hand2_beta/body/meshes/right/r_i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; visual mesh filename=package://wuji_description/hand2_beta/body/meshes/right/r_i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
- link r_index_finger_proximal_abd: geometry collision mesh filename=package://wuji_description/hand2_beta/body/meshes/right/r_i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; visual mesh filename=package://wuji_description/hand2_beta/body/meshes/right/r_i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
- link r_middle_finger_distal: geometry collision mesh filename=package://wuji_description/hand2_beta/body/meshes/right/r_m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; visual mesh filename=package://wuji_description/hand2_beta/body/meshes/right/r_m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
- link r_middle_finger_middle: geometry collision mesh filename=package://wuji_description/hand2_beta/body/meshes/right/r_m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; visual mesh filename=package://wuji_description/hand2_beta/body/meshes/right/r_m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
- link r_middle_finger_proximal: geometry collision mesh filename=package://wuji_description/hand2_beta/body/meshes/right/r_m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; visual mesh filename=package://wuji_description/hand2_beta/body/meshes/right/r_m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
- link r_middle_finger_proximal_abd: geometry collision mesh filename=package://wuji_description/hand2_beta/body/meshes/right/r_m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; visual mesh filename=package://wuji_description/hand2_beta/body/meshes/right/r_m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
- link r_pinky_distal: geometry collision mesh filename=package://wuji_description/hand2_beta/body/meshes/right/r_p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; visual mesh filename=package://wuji_description/hand2_beta/body/meshes/right/r_p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
- link r_pinky_middle: geometry collision mesh filename=package://wuji_description/hand2_beta/body/meshes/right/r_p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; visual mesh filename=package://wuji_description/hand2_beta/body/meshes/right/r_p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
- link r_pinky_proximal: geometry collision mesh filename=package://wuji_description/hand2_beta/body/meshes/right/r_p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; visual mesh filename=package://wuji_description/hand2_beta/body/meshes/right/r_p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
- link r_pinky_proximal_abd: geometry collision mesh filename=package://wuji_description/hand2_beta/body/meshes/right/r_p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; visual mesh filename=package://wuji_description/hand2_beta/body/meshes/right/r_p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
- link r_ring_finger_distal: geometry collision mesh filename=package://wuji_description/hand2_beta/body/meshes/right/r_r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; visual mesh filename=package://wuji_description/hand2_beta/body/meshes/right/r_r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
- link r_ring_finger_middle: geometry collision mesh filename=package://wuji_description/hand2_beta/body/meshes/right/r_r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; visual mesh filename=package://wuji_description/hand2_beta/body/meshes/right/r_r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
- link r_ring_finger_proximal: geometry collision mesh filename=package://wuji_description/hand2_beta/body/meshes/right/r_r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; visual mesh filename=package://wuji_description/hand2_beta/body/meshes/right/r_r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
- link r_ring_finger_proximal_abd: geometry collision mesh filename=package://wuji_description/hand2_beta/body/meshes/right/r_r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; visual mesh filename=package://wuji_description/hand2_beta/body/meshes/right/r_r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
- link r_thumb_distal: geometry collision mesh filename=package://wuji_description/hand2_beta/body/meshes/right/r_t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; visual mesh filename=package://wuji_description/hand2_beta/body/meshes/right/r_t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
- link r_thumb_middle: geometry collision mesh filename=package://wuji_description/hand2_beta/body/meshes/right/r_t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; visual mesh filename=package://wuji_description/hand2_beta/body/meshes/right/r_t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
- link r_thumb_proximal: geometry collision mesh filename=package://wuji_description/hand2_beta/body/meshes/right/r_t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; visual mesh filename=package://wuji_description/hand2_beta/body/meshes/right/r_t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
- link r_thumb_proximal_abd: geometry collision mesh filename=package://wuji_description/hand2_beta/body/meshes/right/r_t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; visual mesh filename=package://wuji_description/hand2_beta/body/meshes/right/r_t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
- link r_wrist: geometry collision mesh filename=package://wuji_description/hand2_beta/body/meshes/right/r_w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; visual mesh filename=package://wuji_description/hand2_beta/body/meshes/right/r_w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
