Commit message: Release v2026.8.14

File: hand2/hand2_beta1/body/urdf/right-ros.urdf (robot description, URDF)
Before this commit: robot wujihand2-right, 26 links, 25 joints
Joints:
- joint r_index_finger_dip: origin xyz=0 0 -0.0295000000000005 rpy=0 0 0 -> xyz=0 0 -0.0295 rpy=0 0 0
- joint r_index_finger_mcp_abd: origin xyz=0 -0.00120098018725688 -0.0145000000001075 rpy=0 0 0 -> xyz=0 -0.001201 -0.0145 rpy=0 0 0
- joint r_index_finger_pip: origin xyz=0 0 -0.0376000000000001 rpy=0 0 0 -> xyz=0 0 -0.0376 rpy=0 0 0
- joint r_middle_finger_dip: origin xyz=0 0 -0.0295000000000004 rpy=0 0 0 -> xyz=0 0 -0.0295 rpy=0 0 0
- joint r_middle_finger_mcp_abd: origin xyz=0 -0.00120098018725689 -0.0145000000001074 rpy=0 0 0 -> xyz=0 -0.001201 -0.0145 rpy=0 0 0
- joint r_middle_finger_pip: origin xyz=0 0 -0.0376000000000002 rpy=0 0 0 -> xyz=0 0 -0.0376 rpy=0 0 0
- joint r_pinky_dip: origin xyz=0 0 -0.0275000000000001 rpy=0 0 0 -> xyz=0 0 -0.0275 rpy=0 0 0
- joint r_pinky_mcp_abd: origin xyz=0 -0.00120098018724169 -0.0145000000001571 rpy=0 0 3.62730676665863E-05 -> xyz=0 -0.001201 -0.0145 rpy=0 0 3.6273E-05
- joint r_pinky_mcp_flex: origin xyz=-0.0373506128592677 -0.000733757744184354 -0.0552962100243675 rpy=-0.029937505027186 0.24885623067687 -0.136021040523522 -> xyz=-0.037351 -0.00073376 -0.055296 rpy=-0.029938 0.24886 -0.13602
- joint r_pinky_pip: origin xyz=0.000100000035494024 0 -0.0335999999999994 rpy=0 0 -3.62730284749225E-05 -> xyz=0.0001 0 -0.0336 rpy=0 0 -3.6273E-05
- joint r_ring_finger_dip: origin xyz=0 0 -0.0295000000000005 rpy=0 0 0 -> xyz=0 0 -0.0295 rpy=0 0 0
- joint r_ring_finger_mcp_abd: origin xyz=0 -0.00120098018725689 -0.0145000000001074 rpy=0 0 0 -> xyz=0 -0.001201 -0.0145 rpy=0 0 0
- joint r_ring_finger_pip: origin xyz=0 0 -0.0376000000000001 rpy=0 0 0 -> xyz=0 0 -0.0376 rpy=0 0 0
- joint r_thumb_cmc_abd: origin xyz=0.000247879062961599 -0.000536579546410674 -0.0147535404706145 rpy=0.205291970332105 0.70050871717831 0.0252378802492596 -> xyz=0.00024788 -0.00053658 -0.014754 rpy=0.20529 0.70051 0.025238
- joint r_thumb_cmc_flex: origin xyz=0.0172096135367909 0.00813796752668306 -0.0164575402574485 rpy=-1.66172905640129 -1.05903134035818 1.99212400148381 -> xyz=0.01721 0.008138 -0.016458 rpy=-1.6617 -1.059 1.9921
- joint r_thumb_ip: origin xyz=-4.99999999923513E-05 0.00385197213324594 -0.0347873872356727 rpy=0.110279740852307 0 0 -> xyz=-5E-05 0 -0.035 rpy=0 0 0
- joint r_thumb_mcp: origin xyz=0 0 -0.032500002798739 rpy=-0.11027974085231 0.0872664625995901 0.567232006897994 -> xyz=0 0 -0.0325 rpy=0 0.087266 0.56723

File: hand2/hand2_beta1/body/urdf/right.urdf (robot description, URDF)
Before this commit: robot wujihand2-right, 26 links, 25 joints
Joints:
- joint r_index_finger_dip: origin xyz=0 0 -0.0295000000000005 rpy=0 0 0 -> xyz=0 0 -0.0295 rpy=0 0 0
- joint r_index_finger_mcp_abd: origin xyz=0 -0.00120098018725688 -0.0145000000001075 rpy=0 0 0 -> xyz=0 -0.001201 -0.0145 rpy=0 0 0
- joint r_index_finger_pip: origin xyz=0 0 -0.0376000000000001 rpy=0 0 0 -> xyz=0 0 -0.0376 rpy=0 0 0
- joint r_middle_finger_dip: origin xyz=0 0 -0.0295000000000004 rpy=0 0 0 -> xyz=0 0 -0.0295 rpy=0 0 0
- joint r_middle_finger_mcp_abd: origin xyz=0 -0.00120098018725689 -0.0145000000001074 rpy=0 0 0 -> xyz=0 -0.001201 -0.0145 rpy=0 0 0
- joint r_middle_finger_pip: origin xyz=0 0 -0.0376000000000002 rpy=0 0 0 -> xyz=0 0 -0.0376 rpy=0 0 0
- joint r_pinky_dip: origin xyz=0 0 -0.0275000000000001 rpy=0 0 0 -> xyz=0 0 -0.0275 rpy=0 0 0
- joint r_pinky_mcp_abd: origin xyz=0 -0.00120098018724169 -0.0145000000001571 rpy=0 0 3.62730676665863E-05 -> xyz=0 -0.001201 -0.0145 rpy=0 0 3.6273E-05
- joint r_pinky_mcp_flex: origin xyz=-0.0373506128592677 -0.000733757744184354 -0.0552962100243675 rpy=-0.029937505027186 0.24885623067687 -0.136021040523522 -> xyz=-0.037351 -0.00073376 -0.055296 rpy=-0.029938 0.24886 -0.13602
- joint r_pinky_pip: origin xyz=0.000100000035494024 0 -0.0335999999999994 rpy=0 0 -3.62730284749225E-05 -> xyz=0.0001 0 -0.0336 rpy=0 0 -3.6273E-05
- joint r_ring_finger_dip: origin xyz=0 0 -0.0295000000000005 rpy=0 0 0 -> xyz=0 0 -0.0295 rpy=0 0 0
- joint r_ring_finger_mcp_abd: origin xyz=0 -0.00120098018725689 -0.0145000000001074 rpy=0 0 0 -> xyz=0 -0.001201 -0.0145 rpy=0 0 0
- joint r_ring_finger_pip: origin xyz=0 0 -0.0376000000000001 rpy=0 0 0 -> xyz=0 0 -0.0376 rpy=0 0 0
- joint r_thumb_cmc_abd: origin xyz=0.000247879062961599 -0.000536579546410674 -0.0147535404706145 rpy=0.205291970332105 0.70050871717831 0.0252378802492596 -> xyz=0.00024788 -0.00053658 -0.014754 rpy=0.20529 0.70051 0.025238
- joint r_thumb_cmc_flex: origin xyz=0.0172096135367909 0.00813796752668306 -0.0164575402574485 rpy=-1.66172905640129 -1.05903134035818 1.99212400148381 -> xyz=0.01721 0.008138 -0.016458 rpy=-1.6617 -1.059 1.9921
- joint r_thumb_ip: origin xyz=-4.99999999923513E-05 0.00385197213324594 -0.0347873872356727 rpy=0.110279740852307 0 0 -> xyz=-5E-05 0 -0.035 rpy=0 0 0
- joint r_thumb_mcp: origin xyz=0 0 -0.032500002798739 rpy=-0.11027974085231 0.0872664625995901 0.567232006897994 -> xyz=0 0 -0.0325 rpy=0 0.087266 0.56723
