Commit message: Release v2026.8.19

File: hand2/hand2_beta1/body/urdf/left-ros.urdf (robot description, URDF)
Before this commit: robot wujihand2-left, 26 links, 25 joints
Links:
- link l_index_finger_distal: geometry collision mesh filename=package://wuji_hand2_beta1_description/meshes/left/l_index_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; visual mesh filename=package://wuji_hand2_beta1_description/meshes/left/l_index_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
- link l_index_finger_middle: geometry collision mesh filename=package://wuji_hand2_beta1_description/meshes/left/l_index_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; visual mesh filename=package://wuji_hand2_beta1_description/meshes/left/l_index_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
- link l_index_finger_proximal: geometry collision mesh filename=package://wuji_hand2_beta1_description/meshes/left/l_index_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; visual mesh filename=package://wuji_hand2_beta1_description/meshes/left/l_index_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
- link l_index_finger_proximal_abd: geometry collision mesh filename=package://wuji_hand2_beta1_description/meshes/left/l_index_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; visual mesh filename=package://wuji_hand2_beta1_description/meshes/left/l_index_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
- link l_middle_finger_distal: geometry collision mesh filename=package://wuji_hand2_beta1_description/meshes/left/l_middle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; visual mesh filename=package://wuji_hand2_beta1_description/meshes/left/l_middle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
- link l_middle_finger_middle: geometry collision mesh filename=package://wuji_hand2_beta1_description/meshes/left/l_middle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; visual mesh filename=package://wuji_hand2_beta1_description/meshes/left/l_middle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
- link l_middle_finger_proximal: geometry collision mesh filename=package://wuji_hand2_beta1_description/meshes/left/l_middle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; visual mesh filename=package://wuji_hand2_beta1_description/meshes/left/l_middle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
- link l_middle_finger_proximal_abd: geometry collision mesh filename=package://wuji_hand2_beta1_description/meshes/left/l_middle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; visual mesh filename=package://wuji_hand2_beta1_description/meshes/left/l_middle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
- link l_pinky_distal: geometry collision mesh filename=package://wuji_hand2_beta1_description/meshes/left/l_pinky_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; visual mesh filename=package://wuji_hand2_beta1_description/meshes/left/l_pinky_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
- link l_pinky_middle: geometry collision mesh filename=package://wuji_hand2_beta1_description/meshes/left/l_pinky_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; visual mesh filename=package://wuji_hand2_beta1_description/meshes/left/l_pinky_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
- link l_pinky_proximal: geometry collision mesh filename=package://wuji_hand2_beta1_description/meshes/left/l_pinky_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; visual mesh filename=package://wuji_hand2_beta1_description/meshes/left/l_pinky_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
- link l_pinky_proximal_abd: geometry collision mesh filename=package://wuji_hand2_beta1_description/meshes/left/l_pinky_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; visual mesh filename=package://wuji_hand2_beta1_description/meshes/left/l_pinky_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
- link l_ring_finger_distal: geometry collision mesh filename=package://wuji_hand2_beta1_description/meshes/left/l_ring_f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; visual mesh filename=package://wuji_hand2_beta1_description/meshes/left/l_ring_f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
- link l_ring_finger_middle: geometry collision mesh filename=package://wuji_hand2_beta1_description/meshes/left/l_ring_f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; visual mesh filename=package://wuji_hand2_beta1_description/meshes/left/l_ring_f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
- link l_ring_finger_proximal: geometry collision mesh filename=package://wuji_hand2_beta1_description/meshes/left/l_ring_f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; visual mesh filename=package://wuji_hand2_beta1_description/meshes/left/l_ring_f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
- link l_ring_finger_proximal_abd: geometry collision mesh filename=package://wuji_hand2_beta1_description/meshes/left/l_ring_f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; visual mesh filename=package://wuji_hand2_beta1_description/meshes/left/l_ring_f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
- link l_thumb_distal: geometry collision mesh filename=package://wuji_hand2_beta1_description/meshes/left/l_thumb_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; visual mesh filename=package://wuji_hand2_beta1_description/meshes/left/l_thumb_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
- link l_thumb_middle: geometry collision mesh filename=package://wuji_hand2_beta1_description/meshes/left/l_thumb_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; visual mesh filename=package://wuji_hand2_beta1_description/meshes/left/l_thumb_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
- link l_thumb_proximal: geometry collision mesh filename=package://wuji_hand2_beta1_description/meshes/left/l_thumb_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; visual mesh filename=package://wuji_hand2_beta1_description/meshes/left/l_thumb_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
- link l_thumb_proximal_abd: geometry collision mesh filename=package://wuji_hand2_beta1_description/meshes/left/l_thumb_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; visual mesh filename=package://wuji_hand2_beta1_description/meshes/left/l_thumb_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
- link l_wrist: geometry collision mesh filename=package://wuji_hand2_beta1_description/meshes/left/l_wrist.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; visual mesh filename=package://wuji_hand2_beta1_description/meshes/left/l_wrist.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

File: hand2/hand2_beta1/body/urdf/left_with_mount-ros.urdf (robot description, URDF)
Before this commit: robot wujihand2-left, 27 links, 26 joints
Links:
- link l_index_finger_distal: geometry collision mesh filename=package://wuji_hand2_beta1_description/meshes/left/l_index_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; visual mesh filename=package://wuji_hand2_beta1_description/meshes/left/l_index_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
- link l_index_finger_middle: geometry collision mesh filename=package://wuji_hand2_beta1_description/meshes/left/l_index_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; visual mesh filename=package://wuji_hand2_beta1_description/meshes/left/l_index_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
- link l_index_finger_proximal: geometry collision mesh filename=package://wuji_hand2_beta1_description/meshes/left/l_index_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; visual mesh filename=package://wuji_hand2_beta1_description/meshes/left/l_index_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
- link l_index_finger_proximal_abd: geometry collision mesh filename=package://wuji_hand2_beta1_description/meshes/left/l_index_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; visual mesh filename=package://wuji_hand2_beta1_description/meshes/left/l_index_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
- link l_middle_finger_distal: geometry collision mesh filename=package://wuji_hand2_beta1_description/meshes/left/l_middle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; visual mesh filename=package://wuji_hand2_beta1_description/meshes/left/l_middle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
- link l_middle_finger_middle: geometry collision mesh filename=package://wuji_hand2_beta1_description/meshes/left/l_middle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; visual mesh filename=package://wuji_hand2_beta1_description/meshes/left/l_middle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
- link l_middle_finger_proximal: geometry collision mesh filename=package://wuji_hand2_beta1_description/meshes/left/l_middle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; visual mesh filename=package://wuji_hand2_beta1_description/meshes/left/l_middle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
- link l_middle_finger_proximal_abd: geometry collision mesh filename=package://wuji_hand2_beta1_description/meshes/left/l_middle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; visual mesh filename=package://wuji_hand2_beta1_description/meshes/left/l_middle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
- link l_mount: geometry collision mesh filename=package://wuji_hand2_beta1_description/meshes/left/l_mount.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; visual mesh filename=package://wuji_hand2_beta1_description/meshes/left/l_mount.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
- link l_pinky_distal: geometry collision mesh filename=package://wuji_hand2_beta1_description/meshes/left/l_pinky_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; visual mesh filename=package://wuji_hand2_beta1_description/meshes/left/l_pinky_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
- link l_pinky_middle: geometry collision mesh filename=package://wuji_hand2_beta1_description/meshes/left/l_pinky_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; visual mesh filename=package://wuji_hand2_beta1_description/meshes/left/l_pinky_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
- link l_pinky_proximal: geometry collision mesh filename=package://wuji_hand2_beta1_description/meshes/left/l_pinky_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; visual mesh filename=package://wuji_hand2_beta1_description/meshes/left/l_pinky_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
- link l_pinky_proximal_abd: geometry collision mesh filename=package://wuji_hand2_beta1_description/meshes/left/l_pinky_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; visual mesh filename=package://wuji_hand2_beta1_description/meshes/left/l_pinky_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
- link l_ring_finger_distal: geometry collision mesh filename=package://wuji_hand2_beta1_description/meshes/left/l_ring_f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; visual mesh filename=package://wuji_hand2_beta1_description/meshes/left/l_ring_f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
- link l_ring_finger_middle: geometry collision mesh filename=package://wuji_hand2_beta1_description/meshes/left/l_ring_f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; visual mesh filename=package://wuji_hand2_beta1_description/meshes/left/l_ring_f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
- link l_ring_finger_proximal: geometry collision mesh filename=package://wuji_hand2_beta1_description/meshes/left/l_ring_f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; visual mesh filename=package://wuji_hand2_beta1_description/meshes/left/l_ring_f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
- link l_ring_finger_proximal_abd: geometry collision mesh filename=package://wuji_hand2_beta1_description/meshes/left/l_ring_f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; visual mesh filename=package://wuji_hand2_beta1_description/meshes/left/l_ring_f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
- link l_thumb_distal: geometry collision mesh filename=package://wuji_hand2_beta1_description/meshes/left/l_thumb_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; visual mesh filename=package://wuji_hand2_beta1_description/meshes/left/l_thumb_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
- link l_thumb_middle: geometry collision mesh filename=package://wuji_hand2_beta1_description/meshes/left/l_thumb_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; visual mesh filename=package://wuji_hand2_beta1_description/meshes/left/l_thumb_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
- link l_thumb_proximal: geometry collision mesh filename=package://wuji_hand2_beta1_description/meshes/left/l_thumb_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; visual mesh filename=package://wuji_hand2_beta1_description/meshes/left/l_thumb_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
- link l_thumb_proximal_abd: geometry collision mesh filename=package://wuji_hand2_beta1_description/meshes/left/l_thumb_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; visual mesh filename=package://wuji_hand2_beta1_description/meshes/left/l_thumb_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
- link l_wrist: geometry collision mesh filename=package://wuji_hand2_beta1_description/meshes/left/l_wrist.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; visual mesh filename=package://wuji_hand2_beta1_description/meshes/left/l_wrist.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

File: hand2/hand2_beta1/body/urdf/right-ros.urdf (robot description, URDF)
Before this commit: robot wujihand2-right, 26 links, 25 joints
Links:
- link r_index_finger_distal: geometry collision mesh filename=package://wuji_hand2_beta1_description/meshes/right/r_index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; visual mesh filename=package://wuji_hand2_beta1_description/meshes/right/r_index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
- link r_index_finger_middle: geometry collision mesh filename=package://wuji_hand2_beta1_description/meshes/right/r_index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; visual mesh filename=package://wuji_hand2_beta1_description/meshes/right/r_index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
- link r_index_finger_proximal: geometry collision mesh filename=package://wuji_hand2_beta1_description/meshes/right/r_index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; visual mesh filename=package://wuji_hand2_beta1_description/meshes/right/r_index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
- link r_index_finger_proximal_abd: geometry collision mesh filename=package://wuji_hand2_beta1_description/meshes/right/r_index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; visual mesh filename=package://wuji_hand2_beta1_description/meshes/right/r_index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
- link r_middle_finger_distal: geometry collision mesh filename=package://wuji_hand2_beta1_description/meshes/right/r_middl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; visual mesh filename=package://wuji_hand2_beta1_description/meshes/right/r_middl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
- link r_middle_finger_middle: geometry collision mesh filename=package://wuji_hand2_beta1_description/meshes/right/r_middl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; visual mesh filename=package://wuji_hand2_beta1_description/meshes/right/r_middl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
- link r_middle_finger_proximal: geometry collision mesh filename=package://wuji_hand2_beta1_description/meshes/right/r_middl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; visual mesh filename=package://wuji_hand2_beta1_description/meshes/right/r_middl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
- link r_middle_finger_proximal_abd: geometry collision mesh filename=package://wuji_hand2_beta1_description/meshes/right/r_middl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; visual mesh filename=package://wuji_hand2_beta1_description/meshes/right/r_middl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
- link r_pinky_distal: geometry collision mesh filename=package://wuji_hand2_beta1_description/meshes/right/r_pinky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; visual mesh filename=package://wuji_hand2_beta1_description/meshes/right/r_pinky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
- link r_pinky_middle: geometry collision mesh filename=package://wuji_hand2_beta1_description/meshes/right/r_pinky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; visual mesh filename=package://wuji_hand2_beta1_description/meshes/right/r_pinky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
- link r_pinky_proximal: geometry collision mesh filename=package://wuji_hand2_beta1_description/meshes/right/r_pinky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; visual mesh filename=package://wuji_hand2_beta1_description/meshes/right/r_pinky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
- link r_pinky_proximal_abd: geometry collision mesh filename=package://wuji_hand2_beta1_description/meshes/right/r_pinky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; visual mesh filename=package://wuji_hand2_beta1_description/meshes/right/r_pinky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
- link r_ring_finger_distal: geometry collision mesh filename=package://wuji_hand2_beta1_description/meshes/right/r_ring_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; visual mesh filename=package://wuji_hand2_beta1_description/meshes/right/r_ring_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
- link r_ring_finger_middle: geometry collision mesh filename=package://wuji_hand2_beta1_description/meshes/right/r_ring_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; visual mesh filename=package://wuji_hand2_beta1_description/meshes/right/r_ring_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
- link r_ring_finger_proximal: geometry collision mesh filename=package://wuji_hand2_beta1_description/meshes/right/r_ring_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; visual mesh filename=package://wuji_hand2_beta1_description/meshes/right/r_ring_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
- link r_ring_finger_proximal_abd: geometry collision mesh filename=package://wuji_hand2_beta1_description/meshes/right/r_ring_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; visual mesh filename=package://wuji_hand2_beta1_description/meshes/right/r_ring_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
- link r_thumb_distal: geometry collision mesh filename=package://wuji_hand2_beta1_description/meshes/right/r_thumb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; visual mesh filename=package://wuji_hand2_beta1_description/meshes/right/r_thumb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
- link r_thumb_middle: geometry collision mesh filename=package://wuji_hand2_beta1_description/meshes/right/r_thumb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; visual mesh filename=package://wuji_hand2_beta1_description/meshes/right/r_thumb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
- link r_thumb_proximal: geometry collision mesh filename=package://wuji_hand2_beta1_description/meshes/right/r_thumb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; visual mesh filename=package://wuji_hand2_beta1_description/meshes/right/r_thumb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
- link r_thumb_proximal_abd: geometry collision mesh filename=package://wuji_hand2_beta1_description/meshes/right/r_thumb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; visual mesh filename=package://wuji_hand2_beta1_description/meshes/right/r_thumb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
- link r_wrist: geometry collision mesh filename=package://wuji_hand2_beta1_description/meshes/right/r_wrist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; visual mesh filename=package://wuji_hand2_beta1_description/meshes/right/r_wrist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

File: hand2/hand2_beta1/body/urdf/right_with_mount-ros.urdf (robot description, URDF)
Before this commit: robot wujihand2-right, 27 links, 26 joints
Links:
- link r_index_finger_distal: geometry collision mesh filename=package://wuji_hand2_beta1_description/meshes/right/r_index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; visual mesh filename=package://wuji_hand2_beta1_description/meshes/right/r_index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
- link r_index_finger_middle: geometry collision mesh filename=package://wuji_hand2_beta1_description/meshes/right/r_index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; visual mesh filename=package://wuji_hand2_beta1_description/meshes/right/r_index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
- link r_index_finger_proximal: geometry collision mesh filename=package://wuji_hand2_beta1_description/meshes/right/r_index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; visual mesh filename=package://wuji_hand2_beta1_description/meshes/right/r_index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
- link r_index_finger_proximal_abd: geometry collision mesh filename=package://wuji_hand2_beta1_description/meshes/right/r_index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; visual mesh filename=package://wuji_hand2_beta1_description/meshes/right/r_index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
- link r_middle_finger_distal: geometry collision mesh filename=package://wuji_hand2_beta1_description/meshes/right/r_middl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; visual mesh filename=package://wuji_hand2_beta1_description/meshes/right/r_middl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
- link r_middle_finger_middle: geometry collision mesh filename=package://wuji_hand2_beta1_description/meshes/right/r_middl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; visual mesh filename=package://wuji_hand2_beta1_description/meshes/right/r_middl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
- link r_middle_finger_proximal: geometry collision mesh filename=package://wuji_hand2_beta1_description/meshes/right/r_middl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; visual mesh filename=package://wuji_hand2_beta1_description/meshes/right/r_middl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
- link r_middle_finger_proximal_abd: geometry collision mesh filename=package://wuji_hand2_beta1_description/meshes/right/r_middl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; visual mesh filename=package://wuji_hand2_beta1_description/meshes/right/r_middl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
- link r_mount: geometry collision mesh filename=package://wuji_hand2_beta1_description/meshes/right/r_mount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; visual mesh filename=package://wuji_hand2_beta1_description/meshes/right/r_mount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
- link r_pinky_distal: geometry collision mesh filename=package://wuji_hand2_beta1_description/meshes/right/r_pinky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; visual mesh filename=package://wuji_hand2_beta1_description/meshes/right/r_pinky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
- link r_pinky_middle: geometry collision mesh filename=package://wuji_hand2_beta1_description/meshes/right/r_pinky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; visual mesh filename=package://wuji_hand2_beta1_description/meshes/right/r_pinky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
- link r_pinky_proximal: geometry collision mesh filename=package://wuji_hand2_beta1_description/meshes/right/r_pinky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; visual mesh filename=package://wuji_hand2_beta1_description/meshes/right/r_pinky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
- link r_pinky_proximal_abd: geometry collision mesh filename=package://wuji_hand2_beta1_description/meshes/right/r_pinky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; visual mesh filename=package://wuji_hand2_beta1_description/meshes/right/r_pinky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
- link r_ring_finger_distal: geometry collision mesh filename=package://wuji_hand2_beta1_description/meshes/right/r_ring_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; visual mesh filename=package://wuji_hand2_beta1_description/meshes/right/r_ring_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
- link r_ring_finger_middle: geometry collision mesh filename=package://wuji_hand2_beta1_description/meshes/right/r_ring_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; visual mesh filename=package://wuji_hand2_beta1_description/meshes/right/r_ring_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
- link r_ring_finger_proximal: geometry collision mesh filename=package://wuji_hand2_beta1_description/meshes/right/r_ring_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; visual mesh filename=package://wuji_hand2_beta1_description/meshes/right/r_ring_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
- link r_ring_finger_proximal_abd: geometry collision mesh filename=package://wuji_hand2_beta1_description/meshes/right/r_ring_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; visual mesh filename=package://wuji_hand2_beta1_description/meshes/right/r_ring_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
- link r_thumb_distal: geometry collision mesh filename=package://wuji_hand2_beta1_description/meshes/right/r_thumb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; visual mesh filename=package://wuji_hand2_beta1_description/meshes/right/r_thumb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
- link r_thumb_middle: geometry collision mesh filename=package://wuji_hand2_beta1_description/meshes/right/r_thumb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; visual mesh filename=package://wuji_hand2_beta1_description/meshes/right/r_thumb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
- link r_thumb_proximal: geometry collision mesh filename=package://wuji_hand2_beta1_description/meshes/right/r_thumb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; visual mesh filename=package://wuji_hand2_beta1_description/meshes/right/r_thumb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
- link r_thumb_proximal_abd: geometry collision mesh filename=package://wuji_hand2_beta1_description/meshes/right/r_thumb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; visual mesh filename=package://wuji_hand2_beta1_description/meshes/right/r_thumb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
- link r_wrist: geometry collision mesh filename=package://wuji_hand2_beta1_description/meshes/right/r_wrist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; visual mesh filename=package://wuji_hand2_beta1_description/meshes/right/r_wrist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
